File: Schematics/RPI.kicad_sch (KiCad schematic)
At the start: 9 parts, among them J1 RPi GPIO, U2 24LC256

Commit message: Added all footprints, updated PCB
Added footprints using uni available components where possible. Might be necessary to change op-amps as they are large and not made for audio. PCB has a mockup of component placements but probably needs expanded.
Parts:
- C9: footprint (none) -> Capacitor_SMD:C_0805_2012Metric_Pad1.18x1.45mm_HandSolder
- R1, R2, R3, R4, R5: footprint Resistor_SMD:R_0603_1608Metric_Pad0.98x0.95mm_HandSolder -> Resistor_SMD:R_0805_2012Metric_Pad1.20x1.40mm_HandSolder
- U2: footprint Package_DIP:DIP-8_W7.62mm_Socket -> Package_SO:SOIC-8_3.9x4.9mm_P1.27mm
Changed lines of the file:
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@@
 			"cQBJAHUAcwBkAHMAcABWAFIAWAByADAAawBXADEAQwB0AGcAcQA5AEIAKwBKAFMAaQAxAEkAVwA4"
 			"AG4AdABDADAAZABpAFUANABTAFIAdQBTADIAbAAxAG8ASQA2AGoAWgBLAHMAbgBxADcAcQAvAG8A"
-			"NQBOAFgAZAArADEAYQBqAA=="
+			"NQBOAFgAZAArADEAYQBqAAAAcQAAAFEAAABNAAAAbAAAAFUAAABDAAAATgAAAEUAAABuAAAATgAA"
+			"AG0AAABPAAAAdAAAADIAAABVAAAAUgAAAHcAAABJAAAAQQAAAHEAAABiAAAAQQAAAEYAAABhAAAA"
+			"egAAAE8AAAAxAAAAVAAAAHIAAABwAAAAZAAAAE4AAABlAAAATgAAADIAAABVAAAANQAAAGIAAAAz"
+			"AAAAaQAAAGgAAAB5AAAANwAAAEoAAABXAAAAQQAAAHYAAABUAAAASgAAACsAAABVAAAAeQAAAEEA"
+			"AABnAAAARQAAAHEAAABvAAAAaAAAADkAAAArAAAAdwAAAFcAAABUAAAAaAAAAGcAAAB3AAAASQAA"
+			"AEEAAABjAAAAVQAAAEgAAABaAAAAQwAAAGMAAAA2AAAAeQAAAHAAAABJAAAAegAAADEAAAAwAAAA"
+			"eAAAAGgAAABEAAAANQAAAEMAAAA5AAAARwAAAEEAAAByAAAAWQAAAGEAAABvAAAAdgAAAG0AAABQ"
+			"AAAARwAAAGoAAABNAAAAbgAAADUAAAArAAAAeAAAAFUAAAByAAAAVgAAAG8AAABoAAAANgAAADkA"
+			"AABlAAAAcAAAAEoAAABCAAAAMgAAAGYAAAB5AAAANQAAAE0AAABuAAAAaQAAAHMAAABzAAAAcwAA"
+			"AHUAAABNAAAAMwAAADcAAABEAAAALwAAAEkAAABCAAAANQAAAEkAAABrAAAAaQAAAHoAAABSAAAA"
+			"aAAAADcAAABXAAAAcQAAAGQAAAB1AAAAcgAAAC8AAAA0AAAAOQAAADcAAABxAAAATgAAADcAAAA5"
+			"AAAAKwAAAEEAAAAxAAAANwAAAEMAAABQAAAAZwAAAEcAAABRAAAASgAAAFIAAABKAAAAaQAAAEkA"
+			"AABoAAAAawAAAFcAAABhAAAANQAAADAAAAAyAAAAcwAAAGwAAAByAAAAawAAAGsAAABPAAAAQQAA"
+			"AFAAAABuAAAAbAAAAHkAAAB4AAAAdAAAAEoAAABQAAAAVAAAADgAAABMAAAAMgAAAG0AAAA1AAAA"
+			"MwAAAGEAAAA1AAAAawAAAGMAAABvAAAAaQAAAFEAAABPAAAAdgAAAEYAAAAxAAAAeAAAAHcAAABn"
+			"AAAAVQAAAEEAAABHAAAAUAAAAHAAAABuAAAAaAAAAE0AAABPAAAAaAAAADMAAAAzAAAAMwAAADIA"
+			"AABuAAAARgAAAE4AAABjAAAANwAAAHQAAABVAAAAMwAAAG4AAABkAAAALwAAAHIAAABrAAAATwAA"
+			"AHQAAABSAAAANAAAAGoAAABSAAAAOAAAAEMAAABGAAAARQAAAHIAAAA2AAAAbwAAAFoAAABmAAAA"
+			"YwAAAGEAAAA2AAAARwAAAA=="
 		)
 	)
@@
 			"RQBXAEwARgBtAEwASwBsAEMAbABLAGMAVQB3AFEAdgBaADQANgBkAGEAcQA0ACsATwBLAEwAcABW"
 			"AFYAaABqAFMATwB6AFAAbgBIAFMAUwBTAGQASgB2AHcASABzAGgASgBMAG8AbwArAHIAZwBGAEYA"
-			"TABDAHEAZwBSAEIAYgB2AHYAbABkAFYATw=="
+			"TABDAHEAZwBSAEIAYgB2AHYAbABkAFYATwAAAAAAAAAAAAAAAAAAAAAAAAAAAAAAAAAAAAAAAAAA"
+			"AAAAAAAAAAAAAAAAAAAAAAAAAAAAAAAAAAAAAAAAAAAAAAAAAAAAAAAAAAAAAAAAAAAAAAAAAAAA"
+			"AAAAAAAAAAAAAAAAAAAAAAAAAAAAAAAAAAAAAAAAAAAAAAAAAAAAAAAAAAAAAAAAAAAAAAAAAAAA"
+			"AAAAAAAAAAAAAAAAAAAAAAAAAAAAAAAAAAAAAAAAAAAAAAAAAAAAAAAAAAAAAAAAAAAAAAAAAAAA"
+			"AAAAAAAAAAAAAAAAAAAAAAAAAAAAAAAAAAAAAAAAAAAAAAAAAAAAAAAAAAAAAAAAAAAAAAAAAAAA"
+			"AAAAAAAAAAAAAAAAAAAAAAAAAAAAAAAAAAAAAAAAAAAAAAAAAAAAAAAAAAAAAAAAAAAAAAAAAAAA"
+			"AAAAAAAAAAAAAAAAAAAAAAAAAAAAAAAAAAAAAAAAAAAAAAAAAAAAAAAAAAAAAAAAAAAAAAAAAAAA"
+			"AAAAAAAAAAAAAAAAAAAAAAAAAAAAAAAAAAAAAAAAAAAAAAAAAAAAAAAAAAAAAAAAAAAAAAAAAAAA"
+			"AAAAAAAAAAAAAAAAAAAAAAAAAAAAAAAAAAAAAAAAAAAAAAAAAAAAAAAAAAAAAAAAAAAAAAAAAAAA"
+			"AAAAAAAAAAAAAAAAAAAAAAAAAAAAAAAAAAAAAAAAAAAAAAAAAAAAAAAAAAAAAAAAAAAAAAAAAAAA"
+			"AAAAAAAAAAAAAAAAAAAAAAAAAAAAAAAAAAAAAAAAAAAAAAAAAAAAAAAAAAAAAAAAAAAAAAAAAAAA"
+			"AAAAAAAAAAAAAAAAAAAAAAAAAAAAAAAAAAAAAAAAAAAAAAAAAAAAAAAAAAAAAAAAAAAAAAAAAAAA"
+			"AAAAAAAAAAAAAAAAAAAAAAAAAAAAAAAAAAAAAAAAAAAAAAAAAAAAAAAAAAAAAAAAAAAAAAAAAAAA"
+			"AAAAAAAAAAAAAAAAAAAAAAAAAAAAAAAAAAAAAAAAAAAAAAAAAAAAAAAAAAAAAAAAAAAAAAAAAAAA"
+			"AAAAAAAAAAAAAAAAAAAAAAAAAAAAAAAAAAAAAAAAAAAAAAAAAAAAAAAAAAAAAAAAAAAAAAAAAAAA"
+			"AAAAAAAAAAAAAAAAAAAAAAAAAAAAAAAAAAAAAAAAAAAAAAAAAAAAAAAAAAAAAAAAAAAAAAAAAAAA"
+			"AAAAAAAAAAAAAAAAAAAAAAAAAAAAAAAAAAAAAAAAAAAAAAAAAAAAAAAAAAAAAAAAAAAAAAAAAAAA"
+			"AAAAAAAAAAAAAAAAAAAAAAAAAAAAAAAAAAAAAAAAAAAAAAAAAAAAAAAAAAAAAAAAAAAAAAAAAAAA"
+			"AAAAAAAAAAAAAAAAAAAAAAAAAAAAAAAAAA=="
 		)
 	)
@@
 			)
 		)
-		(property "Footprint" ""
+		(property "Footprint" "Capacitor_SMD:C_0805_2012Metric_Pad1.18x1.45mm_HandSolder"
 			(at 26.67 54.9148 0)
 			(effects
@@
 			)
 		)
-		(property "Footprint" "Resistor_SMD:R_0603_1608Metric_Pad0.98x0.95mm_HandSolder"
+		(property "Footprint" "Resistor_SMD:R_0805_2012Metric_Pad1.20x1.40mm_HandSolder"
 			(at 45.212 60.96 90)
 			(effects
@@
 			)
 		)
-		(property "Footprint" "Resistor_SMD:R_0603_1608Metric_Pad0.98x0.95mm_HandSolder"
+		(property "Footprint" "Resistor_SMD:R_0805_2012Metric_Pad1.20x1.40mm_HandSolder"
 			(at 24.638 118.11 90)
 			(effects
@@
 			)
 		)
-		(property "Footprint" "Resistor_SMD:R_0603_1608Metric_Pad0.98x0.95mm_HandSolder"
+		(property "Footprint" "Resistor_SMD:R_0805_2012Metric_Pad1.20x1.40mm_HandSolder"
 			(at 24.638 106.68 90)
 			(effects
@@
 			)
 		)
-		(property "Footprint" "Package_DIP:DIP-8_W7.62mm_Socket"
+		(property "Footprint" "Package_SO:SOIC-8_3.9x4.9mm_P1.27mm"
 			(at 35.56 72.39 0)
 			(effects
@@
 			)
 		)
-		(property "Footprint" "Resistor_SMD:R_0603_1608Metric_Pad0.98x0.95mm_HandSolder"
+		(property "Footprint" "Resistor_SMD:R_0805_2012Metric_Pad1.20x1.40mm_HandSolder"
 			(at 71.882 60.96 90)
 			(effects
@@
 			)
 		)
-		(property "Footprint" "Resistor_SMD:R_0603_1608Metric_Pad0.98x0.95mm_HandSolder"
+		(property "Footprint" "Resistor_SMD:R_0805_2012Metric_Pad1.20x1.40mm_HandSolder"
 			(at 49.022 60.96 90)
 			(effects
