File: Schematics/AINPUT.kicad_sch (KiCad schematic)
At the start: 31 parts, among them J2 Line In, J3 Inst In, U3 Opamp_Dual

Commit message: PCB set-up & Jack Sockets
Added 3D file for the Rpi5 and the 1/4" jack sockets. Finalised the dimensions of the PCB with the Pi HAT hole dimensions.
Parts:
- J3: footprint Connector_Audio:Jack_6.35mm_Neutrik_NMJ4HHD2_Horizontal -> custom:NYS2152G
Changed lines of the file:
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@@
 			)
 		)
-		(property "Footprint" "Connector_Audio:Jack_6.35mm_Neutrik_NMJ4HHD2_Horizontal"
+		(property "Footprint" "custom:NYS2152G"
 			(at 104.14 115.57 0)
 			(effects
