File: Schematics/AOUT.kicad_sch (KiCad schematic)
At the start: 25 parts, among them J4 Line Out, J5 Inst Out, Q1 BC547, Q2 BC547, U4 Opamp_Dual

Commit message: PCB set-up & Jack Sockets
Added 3D file for the Rpi5 and the 1/4" jack sockets. Finalised the dimensions of the PCB with the Pi HAT hole dimensions.
Parts:
- J5: footprint Connector_Audio:Jack_6.35mm_Neutrik_NMJ4HHD2_Horizontal -> custom:NYS2152G
Changed lines of the file:
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@@
 			)
 		)
-		(property "Footprint" "Connector_Audio:Jack_6.35mm_Neutrik_NMJ4HHD2_Horizontal"
+		(property "Footprint" "custom:NYS2152G"
 			(at 191.77 127 0)
 			(effects
